Commit message: Minor changes

File: cable-suspended-robots-ros-pkg/urdf/licasa1.urdf.xacro (robot description, xacro)
@@ -101,5 +101,5 @@
   <child link="shoulder_link_x"/>
   <axis xyz="1 0 0"/>
-  <dynamics damping="10.0" friction="0.0"/>
+  <dynamics damping="0.0" friction="0.0"/>
   <limit effort="6.0" lower="${-150/180*pi}" upper="${150/180*pi}" velocity="6"/>
 </joint>
@@ -145,5 +145,5 @@
   <axis xyz="0 1 0"/>
   <dynamics damping="0.0" friction="0.0"/>
-  <limit effort="5000.0" lower="${-90/180*pi}" upper="${90/180*pi}" velocity="6"/>
+  <limit effort="10.0" lower="${-90/180*pi}" upper="${90/180*pi}" velocity="6"/>
 </joint>
 <link name="left_shoulder_roll">
@@ -172,5 +172,5 @@
   <axis xyz="1 0 0"/>
   <dynamics damping="0.0" friction="0.0"/>
-  <limit effort="5000.0" lower="${-50/180*pi}" upper="${90/180*pi}" velocity="6"/>
+  <limit effort="10.0" lower="${-20/180*pi}" upper="${90/180*pi}" velocity="6"/>
 </joint>
 <link name="left_shoulder_yaw">
@@ -199,5 +199,5 @@
   <axis xyz="0 0 1"/>
   <dynamics damping="0.0" friction="0.0"/>
-  <limit effort="5000.0" lower="${-0/180*pi}" upper="${0/180*pi}" velocity="6"/>
+  <limit effort="10.0" lower="${-90/180*pi}" upper="${90/180*pi}" velocity="6"/>
 </joint>
 <link name="left_elbow_pitch">
@@ -254,5 +254,5 @@
   <axis xyz="0 1 0"/>
   <dynamics damping="0.0" friction="0.0"/>
-  <limit effort="5000.0" lower="${-90/180*pi}" upper="${90/180*pi}" velocity="6"/>
+  <limit effort="10.0" lower="${-90/180*pi}" upper="${90/180*pi}" velocity="6"/>
 </joint>
 <link name="right_shoulder_roll">
@@ -281,5 +281,5 @@
   <axis xyz="1 0 0"/>
   <dynamics damping="0.0" friction="0.0"/>
-  <limit effort="5000.0" lower="${-90/180*pi}" upper="${50/180*pi}" velocity="6"/>
+  <limit effort="10.0" lower="${-90/180*pi}" upper="${20/180*pi}" velocity="6"/>
 </joint>
 <link name="right_shoulder_yaw">
@@ -308,5 +308,5 @@
   <axis xyz="0 0 1"/>
   <dynamics damping="0.0" friction="0.0"/>
-  <limit effort="5000.0" lower="${-0/180*pi}" upper="${0/180*pi}" velocity="6"/>
+  <limit effort="10.0" lower="${-90/180*pi}" upper="${90/180*pi}" velocity="6"/>
 </joint>
 <link name="right_elbow_pitch">
@@ -335,5 +335,5 @@
   <axis xyz="0 1 0"/>
   <dynamics damping="0.0" friction="0.0"/>
-  <limit effort="5000.0" lower="${-0/180*pi}" upper="${0/180*pi}" velocity="6"/>
+  <limit effort="10.0" lower="${-150/180*pi}" upper="${150/180*pi}" velocity="6"/>
 </joint>
 <link name="right_forearm_link">
